Commit message: feat: update URDF to rename base link and add odom and base_footprint links with joints

File: go2_robot_sdk/urdf/go2w.urdf (robot description, URDF)
Before this commit: robot go2w, 33 links, 32 joints
Links:
- removed link base
- added link base_footprint
- added link base_link, mass 6.921; collision box size=0.3762 0.0935 0.114; visual mesh filename=package://go2_robot_sdk/dae/go2w_base.dae
- added link map
- added link odom
Joints:
- added joint base_footprint_joint: type fixed, parent base_link, child base_footprint, origin xyz=0 0 0 rpy=0 0 0
- added joint map_joint: type fixed, parent map, child odom, origin xyz=0 0 0 rpy=0 0 0
- added joint odom_joint: type fixed, parent odom, child base_link, origin xyz=0 0 0 rpy=0 0 0
- joint FL_hip_joint: parent base -> base_link
- joint FR_hip_joint: parent base -> base_link
- joint Head_upper_joint: parent base -> base_link
- joint RL_hip_joint: parent base -> base_link
- joint RR_hip_joint: parent base -> base_link
- joint imu_joint: parent base -> base_link
- joint radar_joint: parent base -> base_link
